Commit message: before major changes, robot drives straight only

File: models/robots/basic_colors.urdf.xacro (robot description, xacro)
@@ -1,43 +1,43 @@
 <?xml version="1.0"?>
 <robot>
-  <macro name="Black">
+  <xacro:macro name="Black">
     <material name="black">
       <color rgba="0.0 0.0 0.0 1.0"/>
     </material>
-  </macro>
-  <macro name="Blue">
+  </xacro:macro>
+  <xacro:macro name="Blue">
     <material name="blue">
       <color rgba="0.0 0.0 0.8 1.0"/>
     </material>
-  </macro>
-  <macro name="Green">
+  </xacro:macro>
+  <xacro:macro name="Green">
     <material name="green">
       <color rgba="0.0 0.8 0.0 1.0"/>
     </material>
-  </macro>
-  <macro name="Gray">
+  </xacro:macro>
+  <xacro:macro name="Gray">
     <material name="gray">
       <color rgba="0.7 0.7 0.7 1.0"/>
     </material>
-  </macro>
-  <macro name="DarkGray">
+  </xacro:macro>
+  <xacro:macro name="DarkGray">
     <material name="darkGray">
       <color rgba="0.3 0.3 0.3 1.0"/>
     </material>
-  </macro>
-  <macro name="Red">
+  </xacro:macro>
+  <xacro:macro name="Red">
     <material name="red">
       <color rgba="0.8 0.0 0.0 1.0"/>
     </material>
-  </macro>
-  <macro name="White">
+  </xacro:macro>
+  <xacro:macro name="White">
     <material name="white">
       <color rgba="1.0 1.0 1.0 1.0"/>
     </material>
-  </macro>
-  <macro name="Yellow">
+  </xacro:macro>
+  <xacro:macro name="Yellow">
     <material name="yellow">
       <color rgba="0.8 0.8 0.0 1.0"/>
     </material>
-  </macro>
+  </xacro:macro>
 </robot>

File: models/robots/gvr_base.urdf.xacro (robot description, xacro)
@@ -8,13 +8,13 @@
     <xacro:include filename="$(find gvrbot_simulation)/models/robots/single_wheel.urdf.xacro" />
     <!-- Properties (Constants) -->
-    <property name="M_PI" value="3.14159"/>
-    <property name="base_size_x" value="0.41" /> <!-- Based measured outer dimensions of robot -->
-    <property name="base_size_y" value="0.68" /> <!-- Based measured outer dimensions of robot -->
-    <property name="base_size_z" value="0.16" /> <!-- Based measured outer dimensions of robot -->
-    <property name="base_mass" value="16.92" /> <!-- GvrBot with 4 batteries weighs 39.5 lbs or 17.917 kgs minus 1kg for wheels-->
-    <property name="wheel_radius_big" value="0.085" />
-    <property name="wheel_size_y" value="0.07" />
-    <property name="wheel_mass" value="0.1" />
-    <macro name="gvr_base_macro">
+    <xacro:property name="M_PI" value="3.14159"/>
+    <xacro:property name="base_size_x" value="0.41" /> <!-- Based measured outer dimensions of robot -->
+    <xacro:property name="base_size_y" value="0.68" /> <!-- Based measured outer dimensions of robot -->
+    <xacro:property name="base_size_z" value="0.16" /> <!-- Based measured outer dimensions of robot -->
+    <xacro:property name="base_mass" value="16.92" /> <!-- GvrBot with 4 batteries weighs 39.5 lbs or 17.917 kgs minus 1kg for wheels-->
+    <xacro:property name="wheel_radius_big" value="0.085" />
+    <xacro:property name="wheel_size_y" value="0.07" />
+    <xacro:property name="wheel_mass" value="0.1" />
+    <xacro:macro name="gvr_base_macro">
         <link name="base_link">
             <inertial>
@@ -92,5 +92,4 @@
                 <odometryTopic>/gvr_bot/odom</odometryTopic>
         </plugin>
-        <!--
         <plugin name="p3d_base_controller" filename="libgazebo_ros_p3d.so">
           <alwaysOn>true</alwaysOn>
@@ -115,6 +114,6 @@
           <headingGaussianNoise>0.05</headingGaussianNoise>
         </plugin>
-            -->
+         <!--    -->
         </gazebo>
-    </macro>
+    </xacro:macro>
 </robot>

File: models/robots/inertial_tensors.urdf.xacro (robot description, xacro)
@@ -1,19 +1,19 @@
 <?xml version="1.0"?>
-<robot>
-  <macro name="rectangular_prism_tensor" params="mass len_x len_y len_z">
+<robot xmlns:xacro="http://playerstage.sourceforge.net/gazebo/xmlschema/#xacro">
+  <xacro:macro name="rectangular_prism_tensor" params="mass len_x len_y len_z">
     <inertia   ixx="${ mass / 3 * ( len_y * len_y + len_z * len_z ) }" ixy="${ mass / 4 * len_x * len_y }" ixz="${ mass / 4 * len_x * len_z }"
                iyy="${ mass / 3 * ( len_y * len_y + len_z * len_z ) }" iyz="${ mass / 4 * len_y * len_z }"
                izz="${ mass / 3 * ( len_y * len_y + len_z * len_z ) }" />
-  </macro>
-  <macro name="cuboid_tensor" params="mass len_x len_y len_z">
+  </xacro:macro>
+  <xacro:macro name="cuboid_tensor" params="mass len_x len_y len_z">
     <inertia   ixx="${ mass / 12 * (len_z * len_z + len_y * len_y) }" ixy="0.0" ixz="0.0"
                iyy="${ mass / 12 * (len_z * len_z + len_x * len_x) }" iyz="0.0"
                izz="${ mass / 12 * (len_x * len_x + len_y * len_y) }" />
-  </macro>
+  </xacro:macro>
   <!-- Z axis through the center of top and bottom  -->
-  <macro name="cylinder_tensor" params="mass radius height">
+  <xacro:macro name="cylinder_tensor" params="mass radius height">
     <inertia   ixx="${ mass / 12 * height * height + mass / 4 * radius * radius }" ixy="0.0" ixz="0.0"
                iyy="${ mass / 12 * height * height + mass / 4 * radius * radius }" iyz="0.0"
                izz="${ mass / 2 * radius * radius }" />
-  </macro>
+  </xacro:macro>
 </robot>

File: models/robots/single_wheel.urdf.xacro (robot description, xacro)
@@ -4,5 +4,5 @@
   xmlns:controller="http://playerstage.sourceforge.net/gazebo/xmlschema/#controller"
   xmlns:interface="http://playerstage.sourceforge.net/gazebo/xmlschema/#interface"
-  xmlns:xacro="http://playerstage.sourceforge.net/gazebo/xmlschema/#interface">
+  xmlns:xacro="http://playerstage.sourceforge.net/gazebo/xmlschema/#xacro">
  <xacro:include filename="$(find gvrbot_simulation)/models/robots/inertial_tensors.urdf.xacro" />
   <!-- Properties (Constants) -->
