Commit message: end of cay commit

File: models/robots/gvr_baseV2.urdf.xacro (robot description, xacro)
@@ -4,9 +4,9 @@
     xmlns:interface="http://playerstage.sourceforge.net/gazebo/xmlschema/#interface">
     <xacro:include filename="$(find gvrbot_simulation)/models/robots/inertial_tensors.urdf.xacro" />
-    <xacro:include filename="$(find gvrbot_simulation)/models/robots/single_wheel.urdf.xacro" />
+    <xacro:include filename="$(find gvrbot_simulation)/models/robots/tracked_wheel.urdf.xacro" />
     <!-- Properties (Constants) -->
     <xacro:property name="M_PI" value="3.14159"/>
-    <xacro:property name="base_size_x" value="0.41" /> <!-- Based measured outer dimensions of robot -->
-    <xacro:property name="base_size_y" value="0.68" /> <!-- Based measured outer dimensions of robot -->
+    <xacro:property name="base_size_y" value="0.41" /> <!-- Based measured outer dimensions of robot -->
+    <xacro:property name="base_size_x" value="0.68" /> <!-- Based measured outer dimensions of robot -->
     <xacro:property name="base_size_z" value="0.16" /> <!-- Based measured outer dimensions of robot -->
     <xacro:property name="base_mass" value="16.92" /> <!-- GvrBot with 4 batteries weighs 39.5 lbs or 17.917 kgs minus 1kg for wheels-->
@@ -60,23 +60,22 @@
             </collision>
         </link>
-        <tracked_wheel parent="base_link" prefix="left_0"  offset_y=" 0.25100" offset_x=" ${base_size_x / 2 - 0.04}" offset_z="0" reflect="1" radius="${wheel_radius_big}" height="${wheel_size_y}" mass="${wheel_mass}"/>
-        <tracked_wheel parent="base_link" prefix="left_1"  offset_y=" 0.00000" offset_x=" ${base_size_x / 2 - 0.04}" offset_z="-0.001" reflect="1" radius="${wheel_radius_big}" height="${wheel_size_y}" mass="${wheel_mass}"/>
-        <tracked_wheel parent="base_link" prefix="left_2"  offset_y="-0.25100" offset_x=" ${base_size_x / 2 - 0.04}" offset_z="0" reflect="1" radius="${wheel_radius_big}" height="${wheel_size_y}" mass="${wheel_mass}"/>
-        <tracked_wheel parent="base_link" prefix="left_3"  offset_y=" 0.10550" offset_x=" ${base_size_x / 2 - 0.04}" offset_z="0" reflect="1" radius="${wheel_radius_big}" height="${wheel_size_y}" mass="${wheel_mass}"/>
-        <tracked_wheel parent="base_link" prefix="left_4"  offset_y="-0.10550" offset_x=" ${base_size_x / 2 - 0.04}" offset_z="0" reflect="1" radius="${wheel_radius_big}" height="${wheel_size_y}" mass="${wheel_mass}"/>
-        <tracked_wheel parent="base_link" prefix="left_5"  offset_y=" 0.00500" offset_x=" ${base_size_x / 2 - 0.04}" offset_z="0.001" reflect="1" radius="${wheel_radius_big}" height="${wheel_size_y}" mass="${wheel_mass}"/>
-        <tracked_wheel parent="base_link" prefix="right_0" offset_y=" 0.25100" offset_x="-${base_size_x / 2 - 0.04}" offset_z="0" reflect="1" radius="${wheel_radius_big}" height="${wheel_size_y}" mass="${wheel_mass}"/>
-        <tracked_wheel parent="base_link" prefix="right_1" offset_y=" 0.00000" offset_x="-${base_size_x / 2 - 0.04}" offset_z="-0.001" reflect="1" radius="${wheel_radius_big}" height="${wheel_size_y}" mass="${wheel_mass}"/>
-        <tracked_wheel parent="base_link" prefix="right_2" offset_y="-0.25100" offset_x="-${base_size_x / 2 - 0.04}" offset_z="0" reflect="1" radius="${wheel_radius_big}" height="${wheel_size_y}" mass="${wheel_mass}"/>
-        <tracked_wheel parent="base_link" prefix="right_3" offset_y="-0.10550" offset_x="-${base_size_x / 2 - 0.04}" offset_z="0" reflect="1" radius="${wheel_radius_big}" height="${wheel_size_y}" mass="${wheel_mass}"/>
-        <tracked_wheel parent="base_link" prefix="right_4" offset_y=" 0.10550" offset_x="-${base_size_x / 2 - 0.04}" offset_z="0" reflect="1" radius="${wheel_radius_big}" height="${wheel_size_y}" mass="${wheel_mass}"/>
-        <tracked_wheel parent="base_link" prefix="right_5" offset_y=" 0.00500" offset_x="-${base_size_x / 2 - 0.04}" offset_z="0.001" reflect="1" radius="${wheel_radius_big}" height="${wheel_size_y}" mass="${wheel_mass}"/>
-      <!--  -->
+        <tracked_wheel parent="base_link" prefix="left_0" offset_y=" ${base_size_y / 2 - 0.04}" offset_x=" 0.25100" offset_z="0" reflect="1" wheel_radius="${wheel_radius_big}" wheel_size_y="${wheel_size_y}" mass="${wheel_mass}"/>
+         <!--<tracked_wheel parent="base_link" prefix="left_1" offset_y=" ${base_size_y / 2 - 0.04}" offset_x=" 0.10550" offset_z="0" reflect="1" wheel_radius="${wheel_radius_big}" wheel_size_y="${wheel_size_y}" mass="${wheel_mass}"/>  -->
+        <tracked_wheel parent="base_link" prefix="left_2" offset_y=" ${base_size_y / 2 - 0.04}" offset_x=" 0.00000" offset_z="-0.001" reflect="1" wheel_radius="${wheel_radius_big}" wheel_size_y="${wheel_size_y}" mass="${wheel_mass}"/>
+        <!--<tracked_wheel parent="base_link" prefix="left_3" offset_y=" ${base_size_y / 2 - 0.04}" offset_x="-0.10550" offset_z="0" reflect="1" wheel_radius="${wheel_radius_big}" wheel_size_y="${wheel_size_y}" mass="${wheel_mass}"/>    -->
+        <tracked_wheel parent="base_link" prefix="left_4" offset_y=" ${base_size_y / 2 - 0.04}" offset_x="-0.25100" offset_z="0" reflect="1" wheel_radius="${wheel_radius_big}" wheel_size_y="${wheel_size_y}" mass="${wheel_mass}"/>
+        <tracked_wheel parent="base_link" prefix="right_0" offset_y="-${base_size_y / 2 - 0.04}" offset_x=" 0.25100" offset_z="0" reflect="1" wheel_radius="${wheel_radius_big}" wheel_size_y="${wheel_size_y}" mass="${wheel_mass}"/>
+        <!-- <tracked_wheel parent="base_link" prefix="right_1" offset_y="-${base_size_y / 2 - 0.04}" offset_x=" 0.10550" offset_z="0" reflect="1" wheel_radius="${wheel_radius_big}" wheel_size_y="${wheel_size_y}" mass="${wheel_mass}"/>   -->
+        <tracked_wheel parent="base_link" prefix="right_2" offset_y="-${base_size_y / 2 - 0.04}" offset_x=" 0.00000" offset_z="-0.001" reflect="1" wheel_radius="${wheel_radius_big}" wheel_size_y="${wheel_size_y}" mass="${wheel_mass}"/>
+        <!-- <tracked_wheel parent="base_link" prefix="right_3" offset_y="-${base_size_y / 2 - 0.04}" offset_x="-0.10550" offset_z="0" reflect="1" wheel_radius="${wheel_radius_big}" wheel_size_y="${wheel_size_y}" mass="${wheel_mass}"/>    -->
+        <tracked_wheel parent="base_link" prefix="right_4" offset_y="-${base_size_y / 2 - 0.04}" offset_x="-0.25100" offset_z="0" reflect="1" wheel_radius="${wheel_radius_big}" wheel_size_y="${wheel_size_y}" mass="${wheel_mass}"/>
         <gazebo>
         <plugin name="diffdrive_plugin_multiwheel" filename="libdiffdrive_plugin_multi_wheel.so">
                 <alwaysOn>true</alwaysOn>
-                <updateRate>50.0</updateRate>
-                <leftJoints>left_0_wheel_joint left_1_wheel_joint left_2_wheel_joint left_3_wheel_joint left_4_wheel_joint left_5_wheel_joint</leftJoints>
-                <rightJoints>right_0_wheel_joint right_1_wheel_joint right_2_wheel_joint right_3_wheel_joint right_4_wheel_joint right_5_wheel_joint</rightJoints>
+                <updateRate>10.0</updateRate>
+                <leftJoints>left_0_wheel_joint left_2_wheel_joint left_4_wheel_joint </leftJoints>
+                <rightJoints>right_0_wheel_joint right_2_wheel_joint right_4_wheel_joint </rightJoints>
+                <!-- <leftJoints>left_0_wheel_joint left_1_wheel_joint left_2_wheel_joint left_3_wheel_joint left_4_wheel_joint left_5_wheel_joint</leftJoints>
+                <rightJoints>right_0_wheel_joint right_1_wheel_joint right_2_wheel_joint right_3_wheel_joint right_4_wheel_joint right_5_wheel_joint</rightJoints> -->
                 <wheelSeparation>${base_size_y}</wheelSeparation>
                 <wheelDiameter>${wheel_radius_big*2}</wheelDiameter>
@@ -86,5 +85,5 @@
                 <robotBaseFrame>base_link</robotBaseFrame>
                 <commandTopic>/gvr_bot/cmd_vel</commandTopic>
-                <publishOdometryTf>1</publishOdometryTf>
+                <publishOdometryTf>0</publishOdometryTf>
                 <publishOdometryMsg>1</publishOdometryMsg>
                 <odometryTopic>/gvr_bot/odom</odometryTopic>
@@ -112,5 +111,5 @@
           <headingGaussianNoise>0.05</headingGaussianNoise>
         </plugin>
-         <!--    -->
+        <!--   -->
         </gazebo>
     </xacro:macro>

File: models/robots/gvr_bot.urdf.xacro (robot description, xacro)
@@ -1,9 +1,6 @@
 <?xml version="1.0"?>
 <robot name="gvr_bot"
-    xmlns:xacro="http://playerstage.sourceforge.net/gazebo/xmlschema/#xacro"
-    xmlns:sensor="http://playerstage.sourceforge.net/gazebo/xmlschema/#sensor"
-    xmlns:controller="http://playerstage.sourceforge.net/gazebo/xmlschema/#controller"
-    xmlns:interface="http://playerstage.sourceforge.net/gazebo/xmlschema/#interface">
-    <xacro:include filename="$(find gvrbot_simulation)/models/robots/gvr_base.urdf.xacro" />
+    xmlns:xacro="http://playerstage.sourceforge.net/gazebo/xmlschema/#xacro">
+    <xacro:include filename="$(find gvrbot_simulation)/models/robots/gvr_baseV2.urdf.xacro" />
     <gvr_base_macro />
 </robot>

File: models/robots/model.urdf (robot description, URDF)
Before this commit: robot gvr_bot, 14 links, 13 joints
Links:
- removed link left_1_wheel_link
- removed link left_3_wheel_link
- removed link left_5_wheel_link
- removed link right_1_wheel_link
- removed link right_3_wheel_link
- removed link right_5_wheel_link
- link base_link: geometry collision box size=0.68 0.33 0.085; visual mesh filename=package://gvrbot_simulation/models/meshes/base_linkV4.dae
Joints:
- removed joint left_1_wheel_joint
- removed joint left_3_wheel_joint
- removed joint left_5_wheel_joint
- removed joint right_1_wheel_joint
- removed joint right_3_wheel_joint
- removed joint right_5_wheel_joint
- joint left_0_wheel_joint: axis 1 0 0 -> 0 1 0; origin xyz=0.165 0.251 0 rpy=0 0 0 -> xyz=0.251 0.165 0 rpy=0 0 0
- joint left_2_wheel_joint: axis 1 0 0 -> 0 1 0; origin xyz=0.165 -0.251 0 rpy=0 0 0 -> xyz=0.0 0.165 -0.001 rpy=0 0 0
- joint left_4_wheel_joint: axis 1 0 0 -> 0 1 0; origin xyz=0.165 -0.1055 0 rpy=0 0 0 -> xyz=-0.251 0.165 0 rpy=0 0 0
- joint right_0_wheel_joint: axis 1 0 0 -> 0 1 0; origin xyz=-0.165 0.251 0 rpy=0 0 0 -> xyz=0.251 -0.165 0 rpy=0 0 0
- joint right_2_wheel_joint: axis 1 0 0 -> 0 1 0; origin xyz=-0.165 -0.251 0 rpy=0 0 0 -> xyz=0.0 -0.165 -0.001 rpy=0 0 0
- joint right_4_wheel_joint: axis 1 0 0 -> 0 1 0; origin xyz=-0.165 0.1055 0 rpy=0 0 0 -> xyz=-0.251 -0.165 0 rpy=0 0 0

File: models/robots/single_wheel.urdf.xacro (robot description, xacro)
@@ -1,12 +1,9 @@
 <?xml version="1.0"?>
-<robot
-  xmlns:sensor="http://playerstage.sourceforge.net/gazebo/xmlschema/#sensor"
-  xmlns:controller="http://playerstage.sourceforge.net/gazebo/xmlschema/#controller"
-  xmlns:interface="http://playerstage.sourceforge.net/gazebo/xmlschema/#interface"
-  xmlns:xacro="http://playerstage.sourceforge.net/gazebo/xmlschema/#xacro">
- <xacro:include filename="$(find gvrbot_simulation)/models/robots/inertial_tensors.urdf.xacro" />
-  <!-- Properties (Constants) -->
-  <xacro:property name="M_PI" value="3.14159" />
-  <xacro:macro name="tracked_wheel" params="parent prefix offset_x offset_y offset_z reflect radius height mass">
+<robot xmlns:xacro="http://playerstage.sourceforge.net/gazebo/xmlschema/#xacro">
+    <!-- Included URDF Files -->
+    <xacro:include filename="$(find gvrbot_simulation)/models/robots/inertial_tensors.urdf.xacro" />
+    <!-- Properties (Constants) -->
+    <xacro:property name="M_PI" value="3.14159" />
+    <xacro:macro name="tracked_wheel" params="parent prefix offset_x offset_y offset_z reflect radius height mass">
     <joint name="${prefix}_wheel_joint" type="continuous">
       <origin xyz="${offset_x} ${offset_y * reflect} ${offset_z}" rpy="0 0 0" />
@@ -39,6 +36,6 @@
       </link>
       <gazebo reference="${prefix}_wheel_link" >
-        <mu1>10.0</mu1>
-        <mu2>10.0</mu2>
+        <mu1>1.0</mu1>
+        <mu2>1.0</mu2>
         <kp>1000000.0</kp>
         <kd>100.0</kd>
