Commit message: Aligned the model with center of model, broke physics

File: models/robots/gvr_base.urdf.xacro (robot description, xacro)
@@ -1,5 +1,5 @@
 <?xml version="1.0"?>
-<robot
-    xmlns:xacro="http://playerstage.sourceforge.net/gazebo/xmlschema/#interface"
+<robot name="gvr_bot"
+    xmlns:xacro="http://playerstage.sourceforge.net/gazebo/xmlschema/#xacro"
     xmlns:sensor="http://playerstage.sourceforge.net/gazebo/xmlschema/#sensor"
     xmlns:controller="http://playerstage.sourceforge.net/gazebo/xmlschema/#controller"
@@ -7,49 +7,56 @@
     <xacro:include filename="$(find gvrbot_simulation)/models/robots/inertial_tensors.urdf.xacro" />
     <xacro:include filename="$(find gvrbot_simulation)/models/robots/single_wheel.urdf.xacro" />
-    <xacro:include filename="$(find gvrbot_simulation)/models/robots/basic_colors.urdf.xacro" />
-    <xacro:include filename="$(find gvrbot_simulation)/models/robots/plexiglass_mount.urdf.xacro" />
     <!-- Properties (Constants) -->
     <property name="M_PI" value="3.14159"/>
-    <property name="base_size_x" value="0.380" />
-    <property name="base_size_y" value="0.3" />
-    <property name="base_size_z" value="0.085" />
-    <property name="base_mass" value="25.0" />
+    <property name="base_size_x" value="0.70" />
+    <property name="base_size_y" value="0.25" />
+    <property name="base_size_z" value="0.05" />
+    <property name="base_mass" value="17.92" /> <!-- GvrBot with 4 batteries weighs 39.5 lbs or 17.917 kgs -->
     <property name="wheel_radius_big" value="0.085" />
     <property name="wheel_size_y" value="0.0825" />
     <property name="wheel_mass" value="0.1" />
-    <property name="wheel_offset_z_from_base_link" value="-${wheel_radius_big}" />
+    <!-- <property name="wheel_offset_z_from_base_link" value="-${wheel_radius_big/2}" /> -->
+    <property name="wheel_offset_z_from_base_link" value="0" />
     <macro name="gvr_base_macro">
-        <!-- Links and Joints (i.e., the robot) -->
-        <link name="base_footprint"/>
-        <joint name="bf_to_bl" type="fixed">
-          <origin xyz="0.0 0.0 -${base_size_z * 2}" rpy="0.0 0.0 0.0" />
-          <!--<origin xyz="0.0 0.0 0.0" rpy="0.0 0.0 0.0" />-->
-          <parent link="base_link"/>
-          <child link="base_footprint"/>
-        </joint>
         <link name="base_link">
             <inertial>
                 <mass value="${base_mass}" />
-                <origin xyz="0.0 0.0 0.0" rpy="0 0 0" />
-                <rectangular_prism_tensor mass="${base_mass}" len_x="${base_size_x}" len_y="${base_size_y}" len_z="${base_size_z}" />
+                <origin xyz="0.0 0.0 0.0" rpy="0 0 1.57" />
+                <rectangular_prism_tensor mass="${base_mass}" len_x="${base_size_x+0.10}" len_y="${base_size_y+0.14}" len_z="${base_size_z}" />
             </inertial>
-            <!-- compare the two visual pieces until they match up in size then delete the mesh -->
             <visual>
-                <origin xyz="${base_size_x - 0.05} 0.0 -${base_size_z * 2}" rpy="0 0 1.57" />
+                <origin xyz="0.0 0.0 0.0" rpy="0 0 1.57" />
                 <geometry>
-                    <mesh filename="package://gvrbot_simulation/models/meshes/base_linkV2.dae"/>
+                    <mesh filename="package://gvrbot_simulation/models/meshes/base_linkV3.dae"/>
                 </geometry>
             </visual>
-            <!--visual>
-                <origin xyz="0.0 0.0 -0.085" rpy="0 0 0" />
+            <collision>
+                <origin xyz="0.0 0.0 0.0" rpy="0 0 0" />
                 <geometry>
-                    <box size="${base_size_x} ${base_size_y} ${base_size_z}" />
+                    <box size="${base_size_x} ${base_size_y} ${base_size_z}"/>
                 </geometry>
-                <Green />
-            </visual-->
+            </collision>
+        </link>
+        <joint name="bl_to_bm" type="fixed">
+          <origin xyz="0.0 0.0 0.0" rpy="0.0 0.0 0.0" />
+          <parent link="base_link"/>
+          <child link="base_mark"/>
+        </joint>
+        <link name="base_mark">
+            <inertial>
+                <mass value="0.04" />
+                <origin xyz="0.0 0.0 0.0" rpy="0 0 0" />
+                <rectangular_prism_tensor mass="${base_mass}" len_x="0.02" len_y="0.02" len_z="0.02" />
+            </inertial>
+            <visual>
+                <origin xyz="0.0 0.0 0.0" rpy="0 0 0" />
+                <geometry>
+                    <sphere radius="0.02"/>
+                </geometry>
+            </visual>
             <collision>
-                <origin xyz="0.0 0.0 -0.085" rpy="0 0 0" />
-                <geometry>
-                    <box size="${base_size_x} ${base_size_y} ${base_size_z}" />
+                <origin xyz="0.0 0.0 0.0" rpy="0 0 0.0" />
+                 <geometry>
+                    <sphere radius="0.02"/>
                 </geometry>
             </collision>
@@ -85,4 +92,5 @@
                 <odometryTopic>/gvr_bot/odom</odometryTopic>
         </plugin>
+     <!--
         <plugin name="p3d_base_controller" filename="libgazebo_ros_p3d.so">
           <alwaysOn>true</alwaysOn>
@@ -107,4 +115,5 @@
           <headingGaussianNoise>0.05</headingGaussianNoise>
         </plugin>
+            -->
         </gazebo>
     </macro>

File: models/robots/gvr_bot.urdf.xacro (robot description, xacro)
@@ -1,8 +1,8 @@
 <?xml version="1.0"?>
 <robot name="gvr_bot"
+    xmlns:xacro="http://playerstage.sourceforge.net/gazebo/xmlschema/#xacro"
     xmlns:sensor="http://playerstage.sourceforge.net/gazebo/xmlschema/#sensor"
     xmlns:controller="http://playerstage.sourceforge.net/gazebo/xmlschema/#controller"
-    xmlns:interface="http://playerstage.sourceforge.net/gazebo/xmlschema/#interface"
-    xmlns:xacro="http://www.ros.org/wiki/xacro">
+    xmlns:interface="http://playerstage.sourceforge.net/gazebo/xmlschema/#interface">
     <xacro:include filename="$(find gvrbot_simulation)/models/robots/gvr_base.urdf.xacro" />
     <gvr_base_macro />

File: models/robots/single_wheel.urdf.xacro (robot description, xacro)
@@ -5,5 +5,4 @@
   xmlns:interface="http://playerstage.sourceforge.net/gazebo/xmlschema/#interface"
   xmlns:xacro="http://playerstage.sourceforge.net/gazebo/xmlschema/#interface">
- <xacro:include filename="$(find gvrbot_simulation)/models/robots/basic_colors.urdf.xacro" />
  <xacro:include filename="$(find gvrbot_simulation)/models/robots/inertial_tensors.urdf.xacro" />
   <!-- Properties (Constants) -->
@@ -36,5 +35,4 @@
             <cylinder radius="${radius}" length="${height}" />
           </geometry>
-          <Yellow />
         </visual-->
       </link>

Commit message: corrected physics and inertial tensor, still need to fix wheels

File: models/robots/gvr_base.urdf.xacro (robot description, xacro)
@@ -1,4 +1,4 @@
 <?xml version="1.0"?>
-<robot name="gvr_bot"
+<robot
     xmlns:xacro="http://playerstage.sourceforge.net/gazebo/xmlschema/#xacro"
     xmlns:sensor="http://playerstage.sourceforge.net/gazebo/xmlschema/#sensor"
@@ -9,12 +9,12 @@
     <!-- Properties (Constants) -->
     <property name="M_PI" value="3.14159"/>
-    <property name="base_size_x" value="0.70" />
-    <property name="base_size_y" value="0.25" />
-    <property name="base_size_z" value="0.05" />
-    <property name="base_mass" value="17.92" /> <!-- GvrBot with 4 batteries weighs 39.5 lbs or 17.917 kgs -->
+    <property name="base_size_x" value="0.41" /> <!-- Based measured outer dimensions of robot -->
+    <property name="base_size_y" value="0.68" /> <!-- Based measured outer dimensions of robot -->
+    <property name="base_size_z" value="0.16" /> <!-- Based measured outer dimensions of robot -->
+    <property name="base_mass" value="16.92" /> <!-- GvrBot with 4 batteries weighs 39.5 lbs or 17.917 kgs minus 1kg for wheels-->
     <property name="wheel_radius_big" value="0.085" />
     <property name="wheel_size_y" value="0.0825" />
     <property name="wheel_mass" value="0.1" />
-    <!-- <property name="wheel_offset_z_from_base_link" value="-${wheel_radius_big/2}" /> -->
+    <property name="wheel_offset_z_from_base_link" value="-${wheel_radius_big}" />
     <property name="wheel_offset_z_from_base_link" value="0" />
     <macro name="gvr_base_macro">
@@ -22,17 +22,19 @@
             <inertial>
                 <mass value="${base_mass}" />
-                <origin xyz="0.0 0.0 0.0" rpy="0 0 1.57" />
-                <rectangular_prism_tensor mass="${base_mass}" len_x="${base_size_x+0.10}" len_y="${base_size_y+0.14}" len_z="${base_size_z}" />
-            </inertial>
+                <origin xyz="0.0 -0.1 0.0" rpy="0 0 0" /> <!-- Center of mass on y axis is 10cm in front of the origin
+                <rectangular_prism_tensor mass="${base_mass}" len_x="${base_size_x}" len_y="${base_size_y}" len_z="${base_size_z}" /> -->
+<cuboid_tensor mass="${base_mass}" len_x="${base_size_x}" len_y="${base_size_y}" len_z="${base_size_z}" />
+           </inertial>
             <visual>
-                <origin xyz="0.0 0.0 0.0" rpy="0 0 1.57" />
+                <origin xyz="0.0 0.0 0.0" rpy="0 0 0" />
                 <geometry>
-                    <mesh filename="package://gvrbot_simulation/models/meshes/base_linkV3.dae"/>
+                    <mesh filename="package://gvrbot_simulation/models/meshes/base_linkV4.dae"/>
                 </geometry>
             </visual>
+            <!--   -->
             <collision>
                 <origin xyz="0.0 0.0 0.0" rpy="0 0 0" />
                 <geometry>
-                    <box size="${base_size_x} ${base_size_y} ${base_size_z}"/>
+                    <mesh filename="package://gvrbot_simulation/models/meshes/base_linkV4.dae"/>
                 </geometry>
             </collision>
@@ -43,7 +45,8 @@
           <child link="base_mark"/>
         </joint>
+        <!-- bse_mark is 2cm cube marking the origin of the model and baselink, for use as a reference point -->
         <link name="base_mark">
             <inertial>
-                <mass value="0.04" />
+                <mass value="0.01" />
                 <origin xyz="0.0 0.0 0.0" rpy="0 0 0" />
                 <rectangular_prism_tensor mass="${base_mass}" len_x="0.02" len_y="0.02" len_z="0.02" />
@@ -52,5 +55,5 @@
                 <origin xyz="0.0 0.0 0.0" rpy="0 0 0" />
                 <geometry>
-                    <sphere radius="0.02"/>
+                    <box size="0.02 0.02 0.02"/>
                 </geometry>
             </visual>
@@ -58,8 +61,9 @@
                 <origin xyz="0.0 0.0 0.0" rpy="0 0 0.0" />
                  <geometry>
-                    <sphere radius="0.02"/>
+                    <box size="0.02 0.02 0.02"/>
                 </geometry>
             </collision>
         </link>
+        <!--
         <tracked_wheel parent="base_link" prefix="left_0"  offset_x=" 0.25100" offset_y=" ${base_size_y / 2}" offset_z="${wheel_offset_z_from_base_link}      " reflect="1" radius="${wheel_radius_big}" height="${wheel_size_y}" mass="${wheel_mass}"/>
         <tracked_wheel parent="base_link" prefix="left_1"  offset_x=" 0.00000" offset_y=" ${base_size_y / 2}" offset_z="${wheel_offset_z_from_base_link-0.005}" reflect="1" radius="${wheel_radius_big}" height="${wheel_size_y}" mass="${wheel_mass}"/>
@@ -74,6 +78,7 @@
         <tracked_wheel parent="base_link" prefix="right_4" offset_x=" 0.10550" offset_y="-${base_size_y / 2}" offset_z="${wheel_offset_z_from_base_link}      " reflect="1" radius="${wheel_radius_big}" height="${wheel_size_y}" mass="${wheel_mass}"/>
         <tracked_wheel parent="base_link" prefix="right_5" offset_x=" 0.00500" offset_y="-${base_size_y / 2}" offset_z="${wheel_offset_z_from_base_link+0.005}" reflect="1" radius="${wheel_radius_big}" height="${wheel_size_y}" mass="${wheel_mass}"/>
+        -->
         <gazebo>
-        <!-- TODO: make custom plugin for this that doesn't require an imu -->
+        <!-- TODO: make custom plugin for this that doesn't require an imu
         <plugin name="diffdrive_plugin_multiwheel" filename="libdiffdrive_plugin_multi_wheel.so">
                 <alwaysOn>true</alwaysOn>
@@ -91,6 +96,6 @@
                 <publishOdometryMsg>1</publishOdometryMsg>
                 <odometryTopic>/gvr_bot/odom</odometryTopic>
-        </plugin>
-     <!--
+        </plugin> -->
+        <!--
         <plugin name="p3d_base_controller" filename="libgazebo_ros_p3d.so">
           <alwaysOn>true</alwaysOn>

File: models/robots/inertial_tensors.urdf.xacro (robot description, xacro)
@@ -5,4 +5,9 @@
                iyy="${ mass / 3 * ( len_y * len_y + len_z * len_z ) }" iyz="${ mass / 4 * len_y * len_z }"
                izz="${ mass / 3 * ( len_y * len_y + len_z * len_z ) }" />
+  </macro>
+  <macro name="cuboid_tensor" params="mass len_x len_y len_z">
+    <inertia   ixx="${ mass / 12 * (len_z * len_z + len_y * len_y) }" ixy="0.0" ixz="0.0"
+               iyy="${ mass / 12 * (len_z * len_z + len_x * len_x) }" iyz="0.0"
+               izz="${ mass / 12 * (len_x * len_x + len_y * len_y) }" />
   </macro>
   <!-- Z axis through the center of top and bottom  -->
