Commit message: collision, inertia are much more accurate, robot drives with joy

File: models/robots/gvr_base.urdf.xacro (robot description, xacro)
@@ -14,16 +14,13 @@
     <property name="base_mass" value="16.92" /> <!-- GvrBot with 4 batteries weighs 39.5 lbs or 17.917 kgs minus 1kg for wheels-->
     <property name="wheel_radius_big" value="0.085" />
-    <property name="wheel_size_y" value="0.0825" />
+    <property name="wheel_size_y" value="0.07" />
     <property name="wheel_mass" value="0.1" />
-    <property name="wheel_offset_z_from_base_link" value="-${wheel_radius_big}" />
-    <property name="wheel_offset_z_from_base_link" value="0" />
     <macro name="gvr_base_macro">
         <link name="base_link">
             <inertial>
                 <mass value="${base_mass}" />
-                <origin xyz="0.0 -0.1 0.0" rpy="0 0 0" /> <!-- Center of mass on y axis is 10cm in front of the origin
-                <rectangular_prism_tensor mass="${base_mass}" len_x="${base_size_x}" len_y="${base_size_y}" len_z="${base_size_z}" /> -->
-<cuboid_tensor mass="${base_mass}" len_x="${base_size_x}" len_y="${base_size_y}" len_z="${base_size_z}" />
-           </inertial>
+                <origin xyz="0.0 -0.1 0.0" rpy="0 0 0" /> <!-- Center of mass on y axis is 10cm in front of the origin -->
+                <cuboid_tensor mass="${base_mass}" len_x="${base_size_x}" len_y="${base_size_y}" len_z="${base_size_z}" />
+            </inertial>
             <visual>
                 <origin xyz="0.0 0.0 0.0" rpy="0 0 0" />
@@ -32,12 +29,13 @@
                 </geometry>
             </visual>
-            <!--   -->
             <collision>
-                <origin xyz="0.0 0.0 0.0" rpy="0 0 0" />
+                <origin xyz="0.0 0.0 -0.0085" rpy="0 0 0" />
                 <geometry>
-                    <mesh filename="package://gvrbot_simulation/models/meshes/base_linkV4.dae"/>
+                    <!--  <mesh filename="package://gvrbot_simulation/models/meshes/base_linkV4.dae"/> -->
+                    <box size="${base_size_x} ${base_size_y-0.08} ${base_size_z-0.075}"/>
                 </geometry>
             </collision>
         </link>
+        <!-- base_mark is 2cm cube marking the origin of the model and baselink, for use as a reference point -->
         <joint name="bl_to_bm" type="fixed">
           <origin xyz="0.0 0.0 0.0" rpy="0.0 0.0 0.0" />
@@ -45,8 +43,7 @@
           <child link="base_mark"/>
         </joint>
-        <!-- bse_mark is 2cm cube marking the origin of the model and baselink, for use as a reference point -->
         <link name="base_mark">
             <inertial>
-                <mass value="0.01" />
+                <mass value="0.001" />
                 <origin xyz="0.0 0.0 0.0" rpy="0 0 0" />
                 <rectangular_prism_tensor mass="${base_mass}" len_x="0.02" len_y="0.02" len_z="0.02" />
@@ -65,20 +62,18 @@
             </collision>
         </link>
-        <!--
-        <tracked_wheel parent="base_link" prefix="left_0"  offset_x=" 0.25100" offset_y=" ${base_size_y / 2}" offset_z="${wheel_offset_z_from_base_link}      " reflect="1" radius="${wheel_radius_big}" height="${wheel_size_y}" mass="${wheel_mass}"/>
-        <tracked_wheel parent="base_link" prefix="left_1"  offset_x=" 0.00000" offset_y=" ${base_size_y / 2}" offset_z="${wheel_offset_z_from_base_link-0.005}" reflect="1" radius="${wheel_radius_big}" height="${wheel_size_y}" mass="${wheel_mass}"/>
-        <tracked_wheel parent="base_link" prefix="left_2"  offset_x="-0.25100" offset_y=" ${base_size_y / 2}" offset_z="${wheel_offset_z_from_base_link}      " reflect="1" radius="${wheel_radius_big}" height="${wheel_size_y}" mass="${wheel_mass}"/>
-        <tracked_wheel parent="base_link" prefix="left_3"  offset_x=" 0.10550" offset_y=" ${base_size_y / 2}" offset_z="${wheel_offset_z_from_base_link}      " reflect="1" radius="${wheel_radius_big}" height="${wheel_size_y}" mass="${wheel_mass}"/>
-        <tracked_wheel parent="base_link" prefix="left_4"  offset_x="-0.10550" offset_y=" ${base_size_y / 2}" offset_z="${wheel_offset_z_from_base_link}      " reflect="1" radius="${wheel_radius_big}" height="${wheel_size_y}" mass="${wheel_mass}"/>
-        <tracked_wheel parent="base_link" prefix="left_5"  offset_x=" 0.00500" offset_y=" ${base_size_y / 2}" offset_z="${wheel_offset_z_from_base_link+0.005}" reflect="1" radius="${wheel_radius_big}" height="${wheel_size_y}" mass="${wheel_mass}"/>
-        <tracked_wheel parent="base_link" prefix="right_0" offset_x=" 0.25100" offset_y="-${base_size_y / 2}" offset_z="${wheel_offset_z_from_base_link}      " reflect="1" radius="${wheel_radius_big}" height="${wheel_size_y}" mass="${wheel_mass}"/>
-        <tracked_wheel parent="base_link" prefix="right_1" offset_x=" 0.00000" offset_y="-${base_size_y / 2}" offset_z="${wheel_offset_z_from_base_link-0.005}" reflect="1" radius="${wheel_radius_big}" height="${wheel_size_y}" mass="${wheel_mass}"/>
-        <tracked_wheel parent="base_link" prefix="right_2" offset_x="-0.25100" offset_y="-${base_size_y / 2}" offset_z="${wheel_offset_z_from_base_link}      " reflect="1" radius="${wheel_radius_big}" height="${wheel_size_y}" mass="${wheel_mass}"/>
-        <tracked_wheel parent="base_link" prefix="right_3" offset_x="-0.10550" offset_y="-${base_size_y / 2}" offset_z="${wheel_offset_z_from_base_link}      " reflect="1" radius="${wheel_radius_big}" height="${wheel_size_y}" mass="${wheel_mass}"/>
-        <tracked_wheel parent="base_link" prefix="right_4" offset_x=" 0.10550" offset_y="-${base_size_y / 2}" offset_z="${wheel_offset_z_from_base_link}      " reflect="1" radius="${wheel_radius_big}" height="${wheel_size_y}" mass="${wheel_mass}"/>
-        <tracked_wheel parent="base_link" prefix="right_5" offset_x=" 0.00500" offset_y="-${base_size_y / 2}" offset_z="${wheel_offset_z_from_base_link+0.005}" reflect="1" radius="${wheel_radius_big}" height="${wheel_size_y}" mass="${wheel_mass}"/>
-        -->
+        <tracked_wheel parent="base_link" prefix="left_0"  offset_y=" 0.25100" offset_x=" ${base_size_x / 2 - 0.04}" offset_z="0" reflect="1" radius="${wheel_radius_big}" height="${wheel_size_y}" mass="${wheel_mass}"/>
+        <tracked_wheel parent="base_link" prefix="left_1"  offset_y=" 0.00000" offset_x=" ${base_size_x / 2 - 0.04}" offset_z="-0.001" reflect="1" radius="${wheel_radius_big}" height="${wheel_size_y}" mass="${wheel_mass}"/>
+        <tracked_wheel parent="base_link" prefix="left_2"  offset_y="-0.25100" offset_x=" ${base_size_x / 2 - 0.04}" offset_z="0" reflect="1" radius="${wheel_radius_big}" height="${wheel_size_y}" mass="${wheel_mass}"/>
+        <tracked_wheel parent="base_link" prefix="left_3"  offset_y=" 0.10550" offset_x=" ${base_size_x / 2 - 0.04}" offset_z="0" reflect="1" radius="${wheel_radius_big}" height="${wheel_size_y}" mass="${wheel_mass}"/>
+        <tracked_wheel parent="base_link" prefix="left_4"  offset_y="-0.10550" offset_x=" ${base_size_x / 2 - 0.04}" offset_z="0" reflect="1" radius="${wheel_radius_big}" height="${wheel_size_y}" mass="${wheel_mass}"/>
+        <tracked_wheel parent="base_link" prefix="left_5"  offset_y=" 0.00500" offset_x=" ${base_size_x / 2 - 0.04}" offset_z="0.001" reflect="1" radius="${wheel_radius_big}" height="${wheel_size_y}" mass="${wheel_mass}"/>
+        <tracked_wheel parent="base_link" prefix="right_0" offset_y=" 0.25100" offset_x="-${base_size_x / 2 - 0.04}" offset_z="0" reflect="1" radius="${wheel_radius_big}" height="${wheel_size_y}" mass="${wheel_mass}"/>
+        <tracked_wheel parent="base_link" prefix="right_1" offset_y=" 0.00000" offset_x="-${base_size_x / 2 - 0.04}" offset_z="-0.001" reflect="1" radius="${wheel_radius_big}" height="${wheel_size_y}" mass="${wheel_mass}"/>
+        <tracked_wheel parent="base_link" prefix="right_2" offset_y="-0.25100" offset_x="-${base_size_x / 2 - 0.04}" offset_z="0" reflect="1" radius="${wheel_radius_big}" height="${wheel_size_y}" mass="${wheel_mass}"/>
+        <tracked_wheel parent="base_link" prefix="right_3" offset_y="-0.10550" offset_x="-${base_size_x / 2 - 0.04}" offset_z="0" reflect="1" radius="${wheel_radius_big}" height="${wheel_size_y}" mass="${wheel_mass}"/>
+        <tracked_wheel parent="base_link" prefix="right_4" offset_y=" 0.10550" offset_x="-${base_size_x / 2 - 0.04}" offset_z="0" reflect="1" radius="${wheel_radius_big}" height="${wheel_size_y}" mass="${wheel_mass}"/>
+        <tracked_wheel parent="base_link" prefix="right_5" offset_y=" 0.00500" offset_x="-${base_size_x / 2 - 0.04}" offset_z="0.001" reflect="1" radius="${wheel_radius_big}" height="${wheel_size_y}" mass="${wheel_mass}"/>
+      <!--  -->
         <gazebo>
-        <!-- TODO: make custom plugin for this that doesn't require an imu
         <plugin name="diffdrive_plugin_multiwheel" filename="libdiffdrive_plugin_multi_wheel.so">
                 <alwaysOn>true</alwaysOn>
@@ -96,5 +91,5 @@
                 <publishOdometryMsg>1</publishOdometryMsg>
                 <odometryTopic>/gvr_bot/odom</odometryTopic>
-        </plugin> -->
+        </plugin>
         <!--
         <plugin name="p3d_base_controller" filename="libgazebo_ros_p3d.so">

File: models/robots/single_wheel.urdf.xacro (robot description, xacro)
@@ -13,5 +13,5 @@
       <parent link="${parent}" />
       <child link="${prefix}_wheel_link" />
-      <axis xyz="0 1 0" />
+      <axis xyz="1 0 0" />
       <limit effort="100" velocity="100" />
       <joint_properties damping="0.0" friction="0.0" />
@@ -21,19 +21,20 @@
         <inertial>
           <mass value="${mass}" />
-          <origin xyz=" 0 0 0 " />
+          <origin xyz="0 0 0" rpy="${-M_PI/2} 0 ${-M_PI/2}" /> <!-- Rotate and the cyclinder to use as a wheel -->
           <cylinder_tensor mass="${mass}" radius="${radius}" height="${height}" />
         </inertial>
         <collision>
-          <origin xyz="0 0 0" rpy="${-M_PI/2} 0 0" />
+          <origin xyz="0 0 0" rpy="${-M_PI/2} 0 ${-M_PI/2}" /> <!-- Rotate the cyclinder to use as a wheel -->
           <geometry>
             <cylinder radius="${radius}" length="${height}" />
           </geometry>
         </collision>
-        <!--visual>
-          <origin xyz="0 0 0" rpy="${-M_PI/2} 0 0" />
+<!--
+        <visual>
+          <origin xyz="0 0 0" rpy="${-M_PI/2} 0 ${-M_PI/2}" />
           <geometry>
             <cylinder radius="${radius}" length="${height}" />
           </geometry>
-        </visual-->
+        </visual>  -->
       </link>
       <gazebo reference="${prefix}_wheel_link" >

Commit message: much improved simulation, working with newer diff drive simulation

File: models/robots/gvr_base.urdf.xacro (robot description, xacro)
@@ -4,9 +4,9 @@
     xmlns:interface="http://playerstage.sourceforge.net/gazebo/xmlschema/#interface">
     <xacro:include filename="$(find gvrbot_simulation)/models/robots/inertial_tensors.urdf.xacro" />
-    <xacro:include filename="$(find gvrbot_simulation)/models/robots/single_wheel.urdf.xacro" />
+    <xacro:include filename="$(find gvrbot_simulation)/models/robots/tracked_wheel.urdf.xacro" />
     <!-- Properties (Constants) -->
     <xacro:property name="M_PI" value="3.14159"/>
-    <xacro:property name="base_size_x" value="0.41" /> <!-- Based measured outer dimensions of robot -->
-    <xacro:property name="base_size_y" value="0.68" /> <!-- Based measured outer dimensions of robot -->
+    <xacro:property name="base_size_y" value="0.41" /> <!-- Based measured outer dimensions of robot -->
+    <xacro:property name="base_size_x" value="0.68" /> <!-- Based measured outer dimensions of robot -->
     <xacro:property name="base_size_z" value="0.16" /> <!-- Based measured outer dimensions of robot -->
     <xacro:property name="base_mass" value="16.92" /> <!-- GvrBot with 4 batteries weighs 39.5 lbs or 17.917 kgs minus 1kg for wheels-->
@@ -18,9 +18,9 @@
             <inertial>
                 <mass value="${base_mass}" />
-                <origin xyz="0.0 -0.1 0.0" rpy="0 0 0" /> <!-- Center of mass on y axis is 10cm in front of the origin -->
+                <origin xyz="0.1 0.0 0.0" rpy="0 0 0" /> <!-- Center of mass on x axis is 10cm in front of the origin -->
                 <cuboid_tensor mass="${base_mass}" len_x="${base_size_x}" len_y="${base_size_y}" len_z="${base_size_z}" />
             </inertial>
             <visual>
-                <origin xyz="0.0 0.0 0.0" rpy="0 0 -1.5708" />
+                <origin xyz="0.0 0.0 0.0" rpy="0 0 1.5708" />
                 <geometry>
                     <mesh filename="package://gvrbot_simulation/models/meshes/base_linkV4.dae"/>
@@ -60,34 +60,26 @@
             </collision>
         </link>
-        <tracked_wheel parent="base_link" prefix="left_0"  offset_y=" 0.25100" offset_x=" ${base_size_x / 2 - 0.04}" offset_z="0" reflect="1" radius="${wheel_radius_big}" height="${wheel_size_y}" mass="${wheel_mass}"/>
-        <tracked_wheel parent="base_link" prefix="left_1"  offset_y=" 0.00000" offset_x=" ${base_size_x / 2 - 0.04}" offset_z="-0.001" reflect="1" radius="${wheel_radius_big}" height="${wheel_size_y}" mass="${wheel_mass}"/>
-        <tracked_wheel parent="base_link" prefix="left_2"  offset_y="-0.25100" offset_x=" ${base_size_x / 2 - 0.04}" offset_z="0" reflect="1" radius="${wheel_radius_big}" height="${wheel_size_y}" mass="${wheel_mass}"/>
-        <tracked_wheel parent="base_link" prefix="left_3"  offset_y=" 0.10550" offset_x=" ${base_size_x / 2 - 0.04}" offset_z="0" reflect="1" radius="${wheel_radius_big}" height="${wheel_size_y}" mass="${wheel_mass}"/>
-        <tracked_wheel parent="base_link" prefix="left_4"  offset_y="-0.10550" offset_x=" ${base_size_x / 2 - 0.04}" offset_z="0" reflect="1" radius="${wheel_radius_big}" height="${wheel_size_y}" mass="${wheel_mass}"/>
-        <tracked_wheel parent="base_link" prefix="left_5"  offset_y=" 0.00500" offset_x=" ${base_size_x / 2 - 0.04}" offset_z="0.001" reflect="1" radius="${wheel_radius_big}" height="${wheel_size_y}" mass="${wheel_mass}"/>
-        <tracked_wheel parent="base_link" prefix="right_0" offset_y=" 0.25100" offset_x="-${base_size_x / 2 - 0.04}" offset_z="0" reflect="1" radius="${wheel_radius_big}" height="${wheel_size_y}" mass="${wheel_mass}"/>
-        <tracked_wheel parent="base_link" prefix="right_1" offset_y=" 0.00000" offset_x="-${base_size_x / 2 - 0.04}" offset_z="-0.001" reflect="1" radius="${wheel_radius_big}" height="${wheel_size_y}" mass="${wheel_mass}"/>
-        <tracked_wheel parent="base_link" prefix="right_2" offset_y="-0.25100" offset_x="-${base_size_x / 2 - 0.04}" offset_z="0" reflect="1" radius="${wheel_radius_big}" height="${wheel_size_y}" mass="${wheel_mass}"/>
-        <tracked_wheel parent="base_link" prefix="right_3" offset_y="-0.10550" offset_x="-${base_size_x / 2 - 0.04}" offset_z="0" reflect="1" radius="${wheel_radius_big}" height="${wheel_size_y}" mass="${wheel_mass}"/>
-        <tracked_wheel parent="base_link" prefix="right_4" offset_y=" 0.10550" offset_x="-${base_size_x / 2 - 0.04}" offset_z="0" reflect="1" radius="${wheel_radius_big}" height="${wheel_size_y}" mass="${wheel_mass}"/>
-        <tracked_wheel parent="base_link" prefix="right_5" offset_y=" 0.00500" offset_x="-${base_size_x / 2 - 0.04}" offset_z="0.001" reflect="1" radius="${wheel_radius_big}" height="${wheel_size_y}" mass="${wheel_mass}"/>
-      <!--  -->
-        <gazebo>
-        <plugin name="diffdrive_plugin_multiwheel" filename="libdiffdrive_plugin_multi_wheel.so">
-                <alwaysOn>true</alwaysOn>
-                <updateRate>50.0</updateRate>
-                <leftJoints>left_0_wheel_joint left_1_wheel_joint left_2_wheel_joint left_3_wheel_joint left_4_wheel_joint left_5_wheel_joint</leftJoints>
-                <rightJoints>right_0_wheel_joint right_1_wheel_joint right_2_wheel_joint right_3_wheel_joint right_4_wheel_joint right_5_wheel_joint</rightJoints>
-                <wheelSeparation>${base_size_y}</wheelSeparation>
-                <wheelDiameter>${wheel_radius_big*2}</wheelDiameter>
-                <torque>50000</torque>
-                <interface:position name="position_iface_2"/>
-                <robotNamespace>/</robotNamespace>
-                <robotBaseFrame>base_link</robotBaseFrame>
-                <commandTopic>/gvr_bot/cmd_vel</commandTopic>
-                <publishOdometryTf>1</publishOdometryTf>
-                <publishOdometryMsg>1</publishOdometryMsg>
-                <odometryTopic>/gvr_bot/odom</odometryTopic>
-        </plugin>
+        <tracked_wheel parent="base_link" prefix="left_0" offset_y=" ${base_size_y / 2 - 0.04}" offset_x=" 0.25100" offset_z="0" reflect="1" wheel_radius="${wheel_radius_big}" wheel_size_y="${wheel_size_y}" mass="${wheel_mass}"/>
+        <tracked_wheel parent="base_link" prefix="left_1" offset_y=" ${base_size_y / 2 - 0.04}" offset_x=" 0.10550" offset_z="0" reflect="1" wheel_radius="${wheel_radius_big}" wheel_size_y="${wheel_size_y}" mass="${wheel_mass}"/>
+        <tracked_wheel parent="base_link" prefix="left_2" offset_y=" ${base_size_y / 2 - 0.04}" offset_x=" 0.00000" offset_z="-0.001" reflect="1" wheel_radius="${wheel_radius_big}" wheel_size_y="${wheel_size_y}" mass="${wheel_mass}"/>
+        <tracked_wheel parent="base_link" prefix="left_3" offset_y=" ${base_size_y / 2 - 0.04}" offset_x="-0.10550" offset_z="0" reflect="1" wheel_radius="${wheel_radius_big}" wheel_size_y="${wheel_size_y}" mass="${wheel_mass}"/>
+        <tracked_wheel parent="base_link" prefix="left_4" offset_y=" ${base_size_y / 2 - 0.04}" offset_x="-0.25100" offset_z="0" reflect="1" wheel_radius="${wheel_radius_big}" wheel_size_y="${wheel_size_y}" mass="${wheel_mass}"/>
+        <tracked_wheel parent="base_link" prefix="right_0" offset_y="-${base_size_y / 2 - 0.04}" offset_x=" 0.25100" offset_z="0" reflect="1" wheel_radius="${wheel_radius_big}" wheel_size_y="${wheel_size_y}" mass="${wheel_mass}"/>
+        <tracked_wheel parent="base_link" prefix="right_1" offset_y="-${base_size_y / 2 - 0.04}" offset_x=" 0.10550" offset_z="0" reflect="1" wheel_radius="${wheel_radius_big}" wheel_size_y="${wheel_size_y}" mass="${wheel_mass}"/>
+        <tracked_wheel parent="base_link" prefix="right_2" offset_y="-${base_size_y / 2 - 0.04}" offset_x=" 0.00000" offset_z="-0.001" reflect="1" wheel_radius="${wheel_radius_big}" wheel_size_y="${wheel_size_y}" mass="${wheel_mass}"/>
+        <tracked_wheel parent="base_link" prefix="right_3" offset_y="-${base_size_y / 2 - 0.04}" offset_x="-0.10550" offset_z="0" reflect="1" wheel_radius="${wheel_radius_big}" wheel_size_y="${wheel_size_y}" mass="${wheel_mass}"/>
+        <tracked_wheel parent="base_link" prefix="right_4" offset_y="-${base_size_y / 2 - 0.04}" offset_x="-0.25100" offset_z="0" reflect="1" wheel_radius="${wheel_radius_big}" wheel_size_y="${wheel_size_y}" mass="${wheel_mass}"/>
+      <gazebo>
+      <plugin name="force_based_move_controller" filename="libgazebo_ros_force_based_move.so">
+        <commandTopic>gvr_bot/cmd_vel</commandTopic>
+        <odometryTopic>odom</odometryTopic>
+        <odometryFrame>odom</odometryFrame>
+        <odometryRate>20.0</odometryRate>
+        <robotBaseFrame>base_link</robotBaseFrame>
+        <yaw_velocity_p_gain>500</yaw_velocity_p_gain>
+        <x_velocity_p_gain>3000</x_velocity_p_gain>
+        <y_velocity_p_gain>3000</y_velocity_p_gain>
+        <publishOdometryTf>1</publishOdometryTf>
+      </plugin>
         <plugin name="p3d_base_controller" filename="libgazebo_ros_p3d.so">
           <alwaysOn>true</alwaysOn>
@@ -112,5 +104,5 @@
           <headingGaussianNoise>0.05</headingGaussianNoise>
         </plugin>
-         <!--    -->
+        <!--   -->
         </gazebo>
     </xacro:macro>

File: models/robots/gvr_bot.urdf.xacro (robot description, xacro)
@@ -2,5 +2,5 @@
 <robot name="gvr_bot"
     xmlns:xacro="http://playerstage.sourceforge.net/gazebo/xmlschema/#xacro">
-    <xacro:include filename="$(find gvrbot_simulation)/models/robots/gvr_baseV2.urdf.xacro" />
+    <xacro:include filename="$(find gvrbot_simulation)/models/robots/gvr_base.urdf.xacro" />
     <gvr_base_macro />
 </robot>
